File: circuit/Clock.kicad_sch (KiCad schematic)
At the start: 16 parts, among them SW1 SW_Push, SW2 SW_Push, SW3 SW_Push, SW4 SW_Push, U2 Max98357

Commit message: design sent to mfg
Parts:
- removed ESP32_S1: ~, PaulsCoolKicadLibrary:MODULE_ESP32-S3-ZERO, symbol Pauls Kicad Lib:Waveshare_ESP32_S3_Mini_Zero
- added U1: ESP32_S3_NANO, Paul:ESP32_S3_NANO, symbol Paul:ESP32_S3_NANO
- M1: value ~ -> (none); footprint PaulsCoolKicadLibrary:INMP441 -> Paul:INMP441
Connections:
- net +3V3: now also U1.3V3
- net +5V: now also U1.5V
- net BLCK: now also U1.42
- net CS: now also U1.40
- net Clock: now also U1.21
- net DisplaySignal: now also U1.39
- net GND: now also U1.GND
- net LRCK: now also U1.45
- net MIC_DIN: now also U1.08
- net PhotoresistorSignal: now also U1.15
- net SCK: now also U1.06
- net SPK_DOUT: now also U1.41
- net WS: now also U1.07
- net btnFour: now also U1.10
- net btnOne: now also U1.13
- net btnThree: now also U1.11
- net btnTwo: now also U1.12
- no-connect marks 6 -> 20
Other:
- company: (none) -> TemuWolverine
